Commit message: Updated xacro file

File: bot_description/urdf/bot2.xacro (robot description, xacro)
@@ -43,7 +43,7 @@
   <link name="link_chassis">
     <inertial>
-      <mass value="0.1"/>
+      <mass value="0.02"/>
       <origin rpy="0 0 0" xyz="0 0 0"/>
-      <inertia ixx="0.0004166667" ixy="0" ixz="0" iyy="0.0006666667" iyz="0" izz="0.0004166667"/>
+      <inertia ixx="0.000083333" ixy="0" ixz="0" iyy="0.000133333" iyz="0" izz="0.000083333"/>
     </inertial>
     <!-- body -->
@@ -69,6 +69,8 @@
         <friction>
           <ode>
-            <mu>0.001</mu>
-            <mu2>0.001</mu2>
+            <mu>0</mu>
+            <mu2>0</mu2>
+            <slip1>1000</slip1>
+            <slip2>1000</slip2>
           </ode>
         </friction>
@@ -280,5 +282,5 @@
       <wheelSeparation>0.22</wheelSeparation>
       <wheelDiameter>0.12</wheelDiameter>
-      <wheelTorque>100</wheelTorque>
+      <wheelTorque>10</wheelTorque>
       <commandTopic>cmd_vel</commandTopic>
       <odometryTopic>odom</odometryTopic>
